File: mk18-pcb.kicad_sch (KiCad schematic)
At the start: 49 parts, among them J1 RESET, J10 MACRO-1, J11 MACRO-2, J12 BYPASS MACRO, J13 Fal1-Col-Select, J14 Fal2-Col-Select, J15 Fal1-Row-Select, J16 Fal2-Row-Select, J17 RKJXT-MTX, J18 RKJXT-EC11, J19 Fal2-Col-Select, J2 BYPASS FAL1, J21 Fal2-Col-Select, J3 BYPASS FAL2, J4 BYPASS IND, J5 BYPASS PEDALS, J6 BYPASS SCREEN, J7 Falcon1, J8 Falcon2, J9 PMW JST, U1 TYPE-C-31-M-12, U10 1N4148W_C81598, U11 1N4148W_C81598, U12 1N4148W_C81598, U13 1N4148W_C81598, U14 1N4148W_C81598, U15 1N4148W_C81598, U2 ECT818001569, U3 TYPE-C-31-M-12, U4 74LVC1T45, U4 Pico, U5 TYPE-C-31-M-12, U6 AO3401A_C347476, U7 SRV0504, U9 1N4148W_C81598

Commit message: adding some shift register info and other stuff
Parts:
- added C1, C2, C3, C?: 100nF, footprint:C0402, symbol ct-kicad:C0402X7R104K160NTB
- added P? (x2): FH26W-13S-0_3SHW(60), footprint:FPC-SMD_FH26W-13S-0.3SHW-60, symbol ct-kicad:FH26W-13S-0_3SHW(60)
- added R? (x2): RK73H2ATTD9101F, footprint:R0805, symbol ct-kicad:RK73H2ATTD9101F
- added SW1: SW_SPST, symbol Switch:SW_SPST
- added U16: ECT818001569, kicad-library:FPC-SMD_ECT818001569, symbol kicad-python:ECT818001569
- added U17: 1N4148W, footprint:SOD-123F_L2.7-W1.6-LS3.8-RD, symbol ct-kicad:1N4148W_C81598
- added U8, U?: 74HC595D, footprint:SOIC-16_L9.9-W3.9-P1.27-LS6.0-BL, symbol ct-kicad:74HC595D,118
- added U? (x2): MC74HC589ADR2G, footprint:SOIC-16_L9.9-W3.9-P1.27-LS6.0-BL, symbol ct-kicad:MC74HC589ADR2G
- added U? (x2): 2N7002, footprint:SOT-23-3_L2.9-W1.3-P1.90-LS2.4-BR, symbol ct-kicad:2N7002
- J?: renamed from J17; value RKJXT-MTX -> Conn_01x06_Socket
- J?: renamed from J4; value BYPASS IND -> Conn_01x02_Socket
- J?: renamed from J19; value Fal2-Col-Select -> Conn_02x06_Top_Bottom
- J?: renamed from J7; value Falcon1 -> Conn_01x08_Socket
- J?: renamed from J12; value BYPASS MACRO -> Conn_01x02_Socket
- J?: renamed from J8; value Falcon2 -> Conn_01x08_Socket
- J?: renamed from J11; value MACRO-2 -> Conn_01x06_Socket
- J?: renamed from J1; value RESET -> Conn_01x02_Socket
- J?: renamed from J3; value BYPASS FAL2 -> Conn_01x02_Socket
- J?: renamed from J9; value PMW JST -> Conn_01x06_Socket
- J?: renamed from J10; value MACRO-1 -> Conn_01x06_Socket
- J?: renamed from J15; value Fal1-Row-Select -> Conn_02x07_Top_Bottom
- J?: renamed from J6; value BYPASS SCREEN -> Conn_01x02_Socket
- J?: renamed from J21; value Fal2-Col-Select -> Conn_02x06_Top_Bottom
- J?: renamed from J18; value RKJXT-EC11 -> Conn_01x06_Socket
- J?: renamed from J14; value Fal2-Col-Select -> Conn_02x06_Top_Bottom
- J?: renamed from J5; value BYPASS PEDALS -> Conn_01x02_Socket
- J?: renamed from J16; value Fal2-Row-Select -> Conn_02x07_Top_Bottom
- J?: renamed from J2; value BYPASS FAL1 -> Conn_01x02_Socket
- J?: renamed from J13; value Fal1-Col-Select -> Conn_02x06_Top_Bottom
- U4: value 74LVC1T45 -> SN74LVC1T45DRL; footprint kicad-library:SOT-5X3-6_W1.6-L1.2-P0.50-LS1.6-BL -> Package_TO_SOT_SMD:SOT-563
- renumbered H5 to H?, H3 to H?, H1 to H?, H2 to H?, H4 to H?
Connections:
- net +3V3: now also C1.1, C2.1, C3.1, C?.1, R?.2, R?.2, U8.10 (MasterReset), U8.16 (VCC), U?.10 (MasterReset), U?.16 (VCC), U?.16 (VCC), U?.16 (VCC)
- net GND: now also C1.2, C2.2, C3.2, C?.2, P?.10, P?.6, P?.6, P?.7, P?.7, P?.8, P?.8, P?.9, U16.26, U16.27, U8.13 (OutputEnable), U8.14 (DS), U8.8 (GND), U?.13 (OutputEnable), U?.14 (SA), U?.2 (S), U?.2 (S), U?.8 (GND), U?.8 (GND), U?.8 (GND)
- net VCC: now also P?.2, P?.2, P?.3, P?.3, P?.4, P?.5, U16.13, U16.14, U16.15, U16.16
- net col1: now also U?.1 (B)
- net col2: now also U?.2 (C)
- net col3: now also U?.3 (D)
- net col4: now also U?.4 (E)
- net col5: now also U?.5 (F)
- net col6: now also U?.6 (G)
- net col7: now also U?.7 (H)
- net row1: now also U?.1 (Q1)
- net row2: now also U?.2 (Q2)
- net row3: now also U?.3 (Q3)
- net row4: now also U?.4 (Q4)
- net row5: now also U?.5 (Q5)
- net row6: now also U?.6 (Q6)
- net row7: now also U?.7 (Q7)
- new net: U?.14 (SA), U?.9 (QH)
- new net: U8.9 (Q7S), U?.14 (DS)
- new net: SW1.1 (A), U17.1 (K)
- new net COL_CS: U?.1 (G), U?.10 (OE), U?.10 (OE)
- new net COL_CS_MOS: R?.1, U?.12 (LATCH_CLOCK), U?.12 (LATCH_CLOCK), U?.13 (SLOAD), U?.13 (SLOAD), U?.3 (D)
- new net DI pin: P?.1, P?.1
- new net DO pin: P?.11, P?.11
- new net GND_to_both_bundles: U16.10, U16.11, U16.8, U16.9
- new net MISO: U?.9 (Q7S)
- new net MOSI: U?.9 (QH)
- new net ROW_CS: U8.12 (StorageClock), U?.1 (G), U?.12 (StorageClock)
- new net ROW_CS_MOS: R?.1, U?.3 (D)
- new net Shared_CLK: U8.11 (ShiftClock), U?.11 (SHIFT_CLOCK), U?.11 (SHIFT_CLOCK), U?.11 (ShiftClock)
- new net col pin: P?.10, P?.12, P?.12, P?.4, P?.5, P?.9
- new net col0: SW1.2 (B), U?.15 (A)
- new net col0?_to_both_bundles: U16.6
- new net col10: U?.2 (C)
- new net col11: U?.3 (D)
- new net col12: U?.4 (E)
- new net col13: U?.5 (F)
- new net col14: U?.6 (G)
- new net col15: U?.7 (H)
- new net col1_to_both_bundles: U16.2
- new net col2_to_both_bundles: U16.20
- new net col3_to_both_bundles: U16.21
- new net col4_to_both_bundles: U16.22
- new net col6_to_both_bundles: U16.7
- new net col7_to_both_bundles: U16.25
- new net col8: U?.15 (A)
- new net col9: U?.1 (B)
- new net in_from_keywell_leds: U16.1
- new net out_to_keywell_leds: U16.12
- new net row pin: P?.13, P?.13
- new net row0: U17.2 (A), U?.15 (Q0)
- new net row10: U8.2 (Q2)
- new net row11: U8.3 (Q3)
- new net row12: U8.4 (Q4)
- new net row13: U8.5 (Q5)
- new net row14: U8.6 (Q6)
- new net row15: U8.7 (Q7)
- new net row1_to_thumbs_bundle - as row0: U16.3
- new net row2_to_main_bundle: U16.4
- new net row3_to_main_bundle: U16.18
- new net row4_to_main_bundle: U16.5
- new net row6_to_main_bundle: U16.19
- new net row7_to_main_bundle: U16.23, U16.24
- new net row8: U8.15 (Q0)
- new net row9: U8.1 (Q1)
Other:
- note added: "<----"
- note added: "Column shift registers"
- note added: "Cyboard column pcb?"
- note added: "Cyboard flex-pcb main flex strip"
- note added: "Cyboard single pcb"
- note added: "Example key switch"
- note added: "Flex strip layout: - thumbs on row0, col0-7 - col pcbs on individual tabs"
- note added: "Row shift registers"
- moved on the sheet: U2

Commit message: flipping mosi on cols
Connections:
- net GND: now also U?.9 (QH); no longer U?.14 (SA)
- net MOSI: now also U?.14 (SA); no longer U?.9 (QH)
Changed lines of the file:
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@@
     )
   )
+  (global_label "MOSI" (shape output) (at 590.55 342.9 0) (fields_autoplaced)
+    (effects (font (size 1.27 1.27)) (justify left))
+    (property "Intersheetrefs" "${INTERSHEET_REFS}" (at 598.1314 342.9 0)
+      (effects (font (size 1.27 1.27)) (justify left) hide)
+    )
+  )
   (global_label "row6" (shape input) (at 269.24 335.28 180) (fields_autoplaced)
     (effects (font (size 1.27 1.27)) (justify right))
@@
     )
   )
-  (global_label "MOSI" (shape input) (at 499.11 342.9 180) (fields_autoplaced)
-    (effects (font (size 1.27 1.27)) (justify right))
-    (property "Intersheetrefs" "${INTERSHEET_REFS}" (at 491.5286 342.9 0)
-      (effects (font (size 1.27 1.27)) (justify right) hide)
-    )
-  )
   (global_label "row1" (shape output) (at 223.52 95.25 180) (fields_autoplaced)
     (effects (font (size 1.27 1.27)) (justify right))
@@
     )
   )
+  (symbol (lib_id "power:GND") (at 499.11 342.9 270) (unit 1)
+    (in_bom yes) (on_board yes) (dnp no) (fields_autoplaced)
+    (property "Reference" "#PWR09" (at 492.76 342.9 0)
+      (effects (font (size 1.27 1.27)) hide)
+    )
+    (property "Value" "GND" (at 495.3 342.9 90)
+      (effects (font (size 1.27 1.27)) (justify right))
+    )
+    (property "Footprint" "" (at 499.11 342.9 0)
+      (effects (font (size 1.27 1.27)) hide)
+    )
+    (property "Datasheet" "" (at 499.11 342.9 0)
+      (effects (font (size 1.27 1.27)) hide)
+    )
+    (pin "1")
+    (instances
+      (project "mk18-pcb"
+        (path "/bb2be946-374e-4172-8486-a9a12db7ac7b"
+          (reference "#PWR09") (unit 1)
+        )
+      )
+    )
+  )
   (symbol (lib_id "Connector_Generic:Conn_02x06_Top_Bottom") (at 378.46 45.72 0) (unit 1)
     (in_bom yes) (on_board yes) (dnp no) (fields_autoplaced)
@@
         )
       )
-    )
-  )
-  (symbol (lib_id "power:GND") (at 590.55 342.9 90) (unit 1)
-    (in_bom yes) (on_board yes) (dnp no) (fields_autoplaced)
-    (property "Reference" "#PWR?" (at 596.9 342.9 0)
-      (effects (font (size 1.27 1.27)) hide)
-    )
-    (property "Value" "GND" (at 594.36 342.9 90)
-      (effects (font (size 1.27 1.27)) (justify right))
-    )
-    (property "Footprint" "" (at 590.55 342.9 0)
-      (effects (font (size 1.27 1.27)) hide)
-    )
-    (property "Datasheet" "" (at 590.55 342.9 0)
-      (effects (font (size 1.27 1.27)) hide)
-    )
-    (pin "1")
-    (instances
-      (project "mk18-pcb"
-        (path "/bb2be946-374e-4172-8486-a9a12db7ac7b"
-          (reference "#PWR?") (unit 1)
-        )
-      )

Commit message: cleaning up save state
Connections:
- net GND: now also U?.14 (SA), U?.9 (Q7S); no longer U8.14 (DS), U?.9 (QH)
- net MISO: now also U?.9 (QH); no longer U?.9 (Q7S)
- net MOSI: now also U8.14 (DS); no longer U?.14 (SA)
Other:
- moved on the sheet: SW1, U17

Commit message: capturing updates for the day
Connections:
- net GND: no longer U8.13 (OutputEnable), U?.13 (OutputEnable)
- net ROW_CS: now also U8.13 (OutputEnable), U?.13 (OutputEnable); no longer U8.12 (StorageClock), U?.12 (StorageClock)
- net ROW_CS_MOS: now also U8.12 (StorageClock), U?.12 (StorageClock)
Other:
- moved on the sheet: R?, SW1, U17, U?

Commit message: work from the 31st
Parts:
- removed R?: RK73H2ATTD9101F, footprint:R0805, symbol ct-kicad:RK73H2ATTD9101F
- removed SW1: SW_SPST, symbol Switch:SW_SPST
- removed U17: 1N4148W, footprint:SOD-123F_L2.7-W1.6-LS3.8-RD, symbol ct-kicad:1N4148W_C81598
- removed U?: 2N7002, footprint:SOT-23-3_L2.9-W1.3-P1.90-LS2.4-BR, symbol ct-kicad:2N7002
- added P1, P2, P3, P4, P5, P6, P7, P8, P9: FH26W-13S-0_3SHW(60), footprint:FPC-SMD_FH26W-13S-0.3SHW-60, symbol ct-kicad:FH26W-13S-0_3SHW(60)
- added U17, U18: HC-FPC-05-10-16RLTAG, footprint:FPC-SMD_16P-P0.50_HCTL_HC-FPC-05-10-16RLTAG, symbol ct-kicad:HC-FPC-05-10-16RLTAG
Connections:
- net ROW_CS_MOS is gone; now on net ROW_CS: U8.12 (StorageClock), U?.12 (StorageClock)
- net pmw-miso is gone; now on net SPI1_MISO: J?.8 (Pin_8), U4.16 (GPIO12)
- net pmw-mosi-row9 is gone; now on net SPI1_MOSI: J?.10 (Pin_10), U4.15 (GPIO11)
- net pmw-sck-row8 is gone; now on net SPI1_CLK: J?.12 (Pin_12), J?.2 (Pin_2), U4.14 (GPIO10)
- net COL_CS: now also U4.12 (GPIO9)
- net DI pin: now also P1.1
- net DO pin: now also P1.11
- net GND: now also U4.13 (GND), U4.23 (GND), U4.8 (GND), U8.13 (OutputEnable), U?.13 (OutputEnable), P1.10, P1.6, P1.7, P1.8, P1.9, P2.10, P2.6, P2.7, P2.8, P2.9, P3.10, P3.6, P3.7, P3.8, P3.9, P4.10, P4.6, P4.7, P4.8, P4.9, P5.10, P5.6, P5.7, P5.8, P5.9, P6.10, P6.6, P6.7, P6.8, P6.9, P7.10, P7.6, P7.7, P7.8, P7.9, P8.10, P8.6, P8.7, P8.8, P8.9, P9.10, P9.6, P9.7, P9.8, P9.9, U17.13, U17.14, U17.15, U17.16, U18.13, U18.14, U18.15, U18.16
- net ROW_CS: now also U4.7 (GPIO5); no longer U8.13 (OutputEnable), U?.13 (OutputEnable)
- net VCC: now also P1.2, P1.3, P1.4, P1.5, P2.2, P2.3, P2.4, P2.5, P3.2, P3.3, P3.4, P3.5, P4.2, P4.3, P4.4, P4.5, P5.2, P5.3, P5.4, P5.5, P6.2, P6.3, P6.4, P6.5, P7.2, P7.3, P7.4, P7.5, P8.2, P8.3, P8.4, P8.5, P9.2, P9.3, P9.4, P9.5, U17.1, U17.2, U17.3, U17.4, U18.1, U18.2, U18.3, U18.4
- net col pin: now also P1.12
- net col0: now also U2.2
- net col1: now also U2.20; no longer U2.2, U4.21 (GPIO16)
- net col10: now also P6.12, P7.12, U17.7, U18.7
- net col11: now also P8.12, P9.12, U17.8, U18.8
- net col2: now also U2.21; no longer U2.20, U4.22 (GPIO17)
- net col3: now also U2.22; no longer U2.21, U4.24 (GPIO18)
- net col4: now also U2.17; no longer U2.22, U4.25 (GPIO19)
- net col5: now also U2.7; no longer U2.17, U4.26 (GPIO20)
- net col6: now also U2.6; no longer U2.7, U4.27 (GPIO21)
- net col8: now also P2.12, P3.12, U17.5, U18.5
- net col9: now also P4.12, P5.12, U17.6, U18.6
- net rkjxt-r1: now also U4.10 (GPIO7); no longer U4.12 (GPIO9)
- net rkjxt-r2: now also U4.11 (GPIO8); no longer U4.29 (GPIO22)
- net row pin: now also P1.13
- net row0: now also U2.3
- net row1: now also U2.4; no longer U2.3, U4.4 (GPIO2)
- net row2: now also U2.18; no longer U2.4, U4.5 (GPIO3)
- net row3: now also U2.5; no longer U2.18, U4.6 (GPIO4)
- net row4: now also U2.23; no longer U2.5, U4.7 (GPIO5)
- net row5: now also U2.19; no longer U2.23, U4.9 (GPIO6)
- net row6: now also U2.24; no longer U2.19, U4.10 (GPIO7)
- net row7: no longer U2.24, U4.11 (GPIO8)
- net row8: now also P2.13, P4.13, P6.13, P8.13, U17.9, U18.9
- net row9: now also P3.13, P5.13, P7.13, P9.13, U17.10, U18.10
- net MISO renamed SPI1_MISO
- net MOSI renamed SPI1_MOSI
- net Shared_CLK renamed SPI1_CLK
- net pmw-cs renamed PMW_CS
- new net: P2.1, U17.11
- new net: P2.11, P4.1
- new net: P4.11, P6.1
- new net: P6.11, P8.1
- new net: P5.11, P7.1
- new net: P7.11, P9.1
- new net: P3.11, P5.1
- new net LED_DI_MACRO: U18.11
- new net LED_DO_MACRO: P9.11, U17.12, U18.12
- new net from_row_9_DO: P3.1, P8.11
- no-connect marks 25 -> 47
Other:
- note added: "Macropad Cyboard expander FFC 0.5mm 16-pin to 8x 0.3mm 13-pin"
- note removed: "Example key switch"
- moved on the sheet: C1, C2, C3, C?, J?, P?, R?, U16, U2, U8, U?

Commit message: jan2 updates, relocating shift registers
Parts:
- removed J? (x2): Conn_02x06_Top_Bottom, Connector_PinSocket_2.54mm:PinSocket_2x06_P2.54mm_Vertical, symbol Connector_Generic:Conn_02x06_Top_Bottom
- removed J? (x2): Conn_01x08_Socket, Connector_JST:JST_XH_B8B-XH-A_1x08_P2.50mm_Vertical, symbol Connector:Conn_01x08_Socket
- removed J?: Conn_01x06_Socket, Connector_JST:JST_XH_B6B-XH-A_1x06_P2.50mm_Vertical, symbol Connector:Conn_01x06_Socket
- removed J? (x2): Conn_01x02_Socket, Connector_JST:JST_EH_B2B-EH-A_1x02_P2.50mm_Vertical, symbol Connector:Conn_01x02_Socket
- added FAL1, FAL2, IND1, PWM1: Conn_01x08_Socket, Connector_JST:JST_XH_B8B-XH-A_1x08_P2.50mm_Vertical, symbol Connector:Conn_01x08_Socket
- BOOST-CONVERT1: renamed from U7; footprint kicad-library:SOT-23-6_L2.9-W1.6-P0.95-LS2.8-BL -> ct-kicad:SOT-23-6_L2.9-W1.6-P0.95-LS2.8-BL
- C1, C2, C3: footprint footprint:C0402 -> ct-kicad:C0402
- C4: renamed from C?; footprint footprint:C0402 -> ct-kicad:C0402
- COL_CS_MOS1: renamed from U?; footprint footprint:SOT-23-3_L2.9-W1.3-P1.90-LS2.4-BR -> ct-kicad:SOT-23-3_L2.9-W1.3-P1.90-LS2.4-BR
- CYBOARD-MACRO1: renamed from U18; footprint footprint:FPC-SMD_16P-P0.50_HCTL_HC-FPC-05-10-16RLTAG -> ct-kicad:FPC-SMD_16P-P0.50_HCTL_HC-FPC-05-10-16RLTAG
- CYBOARD-MAIN1: renamed from U2; footprint kicad-library:FPC-SMD_ECT818001569 -> ct-kicad:FPC-SMD_ECT818001569
- D1: footprint kicad-library:SOD-123FL_L2.8-W1.8-LS3.7-BI -> ct-kicad:SOD-123FL_L2.8-W1.8-LS3.7-BI
- F1: footprint kicad-library:F1206 -> ct-kicad:F1206
- J10, J17, J18, J19, J20, J7, J8, J9: renamed from J?; now not fitted; now left out of the parts list
- L1: footprint kicad-library:L0805 -> ct-kicad:L0805
- MOSFET1: renamed from U6; footprint kicad-library:SOT-23_L2.9-W1.3-P1.90-LS2.4-BR -> ct-kicad:SOT-23_L2.9-W1.3-P1.90-LS2.4-BR
- P1: now not fitted
- P10, P11: renamed from P?; now not fitted
- P2, P3, P4, P5, P6, P7, P8, P9, U1, U10, U11, U12, U13, U14, U15, U16, U17, U9: now not fitted; now left out of the parts list
- R1, R2, R3, R4, R5, R6: footprint kicad-library:R0805 -> ct-kicad:R0805
- R7: renamed from R?; footprint footprint:R0805 -> ct-kicad:R0805
- REG-COL1, REG-COL2, REG-ROW2: renamed from U?; footprint footprint:SOIC-16_L9.9-W3.9-P1.27-LS6.0-BL -> ct-kicad:SOIC-16_L9.9-W3.9-P1.27-LS6.0-BL
- REG-ROW1: renamed from U8; footprint footprint:SOIC-16_L9.9-W3.9-P1.27-LS6.0-BL -> ct-kicad:SOIC-16_L9.9-W3.9-P1.27-LS6.0-BL
- SCREEN1: renamed from U3; footprint kicad-library:USB-C_SMD-TYPE-C-31-M-12 -> ct-kicad:USB-C_SMD-TYPE-C-31-M-12
- SPLIT-USB1: renamed from U5; footprint kicad-library:USB-C_SMD-TYPE-C-31-M-12 -> ct-kicad:USB-C_SMD-TYPE-C-31-M-12
- U4: footprint Package_TO_SOT_SMD:SOT-563 -> ct-kicad:SOT-563_L1.6-W1.2-P0.50-LS1.6-BR
- gave numbers to parts that had none: 10
- renumbered U4 to PICO1
Connections:
- net LED_DI_MACRO is gone; now on net LED_KEYS_DO: CYBOARD-MACRO1.11
- net +3V3: now also PWM1.1 (Pin_1)
- net COL_CS: now also PICO1.7 (GPIO5); no longer PICO1.12 (GPIO9)
- net GND: now also SCREEN1.0 (SH), SPLIT-USB1.0 (SH), FAL1.1 (Pin_1), FAL2.1 (Pin_1), IND1.1 (Pin_1), PWM1.7 (Pin_7)
- net LED_DO_MACRO: no longer CYBOARD-MACRO1.12
- net LED_FAL1_DI: now also CYBOARD-MACRO1.12, FAL1.3 (Pin_3)
- net LED_FAL1_DO: now also FAL1.4 (Pin_4), FAL2.3 (Pin_3)
- net LED_FAL2_DO: now also FAL2.4 (Pin_4), IND1.4 (Pin_4)
- net LED_INDICATORS_DO: now also SCREEN1.A6 (DP1), IND1.3 (Pin_3); no longer U1.A6 (DP1)
- net LED_PEDALS_DO: no longer SCREEN1.A6 (DP1)
- net PMW_CS: now also PWM1.5 (Pin_5)
- net ROW_CS: now also PICO1.12 (GPIO9); no longer PICO1.7 (GPIO5)
- net SHIELD: no longer SCREEN1.0 (SH), SPLIT-USB1.0 (SH)
- net SPI1_CLK: now also PWM1.4 (Pin_4)
- net SPI1_MISO: now also PWM1.2 (Pin_2)
- net SPI1_MOSI: now also PWM1.3 (Pin_3)
- net VCC: now also FAL1.2 (Pin_2), FAL2.2 (Pin_2), IND1.2 (Pin_2)
- net fal1-col: now also FAL1.6 (Pin_6)
- net fal1-r1: now also PICO1.24 (GPIO18), FAL1.7 (Pin_7); no longer PICO1.19 (GPIO14)
- net fal1-r2: now also PICO1.25 (GPIO19), FAL1.8 (Pin_8); no longer PICO1.20 (GPIO15)
- net fal1-row: now also FAL1.5 (Pin_5)
- net fal2-col: now also FAL2.6 (Pin_6)
- net fal2-r1: now also PICO1.26 (GPIO20), FAL2.7 (Pin_7); no longer PICO1.32 (GPIO27_ADC1)
- net fal2-r2: now also PICO1.27 (GPIO21), FAL2.8 (Pin_8); no longer PICO1.31 (GPIO26_ADC0)
- net fal2-row: now also FAL2.5 (Pin_5)
- net rkjxt-r1: no longer PICO1.10 (GPIO7)
- net rkjxt-r2: no longer PICO1.11 (GPIO8)
- new net LED_PEDALS_DI: U1.A6 (DP1)
- no-connect marks 47 -> 45
Other:
- note added: "Cyboard flex-pcb main 25-pin connector"
- note added: "Indicators"
- note added: "LED DI-DO bypass jumpers"
- note added: "MCU headers"
- note added: "Peripheral devices"
- note added: "To Macropad Cyboard expander"
- note removed: "<----"
- note removed: "Cyboard flex-pcb keys connector"
- note removed: "LED DI-DO loopies"
- moved on the sheet: C1, C2, C3, C4, COL_CS_MOS1, CYBOARD-MACRO1, CYBOARD-MAIN1, H1, H2, H3, H4, H5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

Commit message: getting ready to re-do the shift register routing so we can have pinouts.
Parts:
- added C5, C6: 100nF, ct-kicad:C0402, symbol ct-kicad:C0402X7R104K160NTB
- added COL1, COL2, ROW1, ROW2: Conn_01x08_Socket, Connector_JST:JST_XH_B8B-XH-A_1x08_P2.50mm_Vertical, symbol Connector:Conn_01x08_Socket
- added LED-EXT-DO1: Conn_01x02_Socket, Connector_JST:JST_EH_B2B-EH-A_1x02_P2.50mm_Vertical, symbol Connector:Conn_01x02_Socket
Connections:
- net +3V3: now also C5.1
- net GND: now also C5.2, C6.2
- net LED_INDICATORS_DO: now also SCREEN1.B6 (DP2)
- net VCC: now also C6.1
- net col0: now also COL1.1 (Pin_1)
- net col1: now also COL1.2 (Pin_2)
- net col10: now also COL2.3 (Pin_3)
- net col11: now also COL2.4 (Pin_4)
- net col12: now also COL2.5 (Pin_5)
- net col13: now also COL2.6 (Pin_6)
- net col14: now also COL2.7 (Pin_7)
- net col15: now also COL2.8 (Pin_8)
- net col2: now also COL1.3 (Pin_3)
- net col3: now also COL1.4 (Pin_4)
- net col4: now also COL1.5 (Pin_5)
- net col5: now also COL1.6 (Pin_6)
- net col6: now also COL1.7 (Pin_7)
- net col7: now also COL1.8 (Pin_8)
- net col8: now also COL2.1 (Pin_1)
- net col9: now also COL2.2 (Pin_2)
- net row0: now also ROW1.1 (Pin_1)
- net row1: now also ROW1.2 (Pin_2)
- net row10: now also ROW2.3 (Pin_3)
- net row11: now also ROW2.4 (Pin_4)
- net row12: now also ROW2.5 (Pin_5)
- net row13: now also ROW2.6 (Pin_6)
- net row14: now also ROW2.7 (Pin_7)
- net row15: now also ROW2.8 (Pin_8)
- net row2: now also ROW1.3 (Pin_3)
- net row3: now also ROW1.4 (Pin_4)
- net row4: now also ROW1.5 (Pin_5)
- net row5: now also ROW1.6 (Pin_6)
- net row6: now also ROW1.7 (Pin_7)
- net row7: now also ROW1.8 (Pin_8)
- net row8: now also ROW2.1 (Pin_1)
- net row9: now also ROW2.2 (Pin_2)
- net LED_SCREEN_DO: now reaches SCREEN1.A7 (DN1)
- net LED_SCREEN_DO: now also SCREEN1.B7 (DN2), LED-EXT-DO1.1 (Pin_1)
- no-connect marks 45 -> 42

Commit message: jan4 updates
Parts:
- removed BOOST-CONVERT1: SRV0504, ct-kicad:SOT-23-6_L2.9-W1.6-P0.95-LS2.8-BL, symbol kicad-symbols:SRV0504
- added U2: AZC199-04S-MS, ct-kicad:TSOT-23-6_L2.9-W1.6-P0.95-LS2.8-BL, symbol ct-kicad:AZC199-04S-MS
Connections:
- net +3V3: now also PWM1.6 (Pin_6); no longer PWM1.1 (Pin_1)
- net GND: now also PWM1.1 (Pin_1), U2.2; no longer PWM1.7 (Pin_7)
- net Serial_VBUS: now also SCREEN1.A4 (VBUS), SCREEN1.A9 (VBUS), SCREEN1.B4 (VBUS), SCREEN1.B9 (VBUS)
- net Split_Comms_RX-A7: now also U2.1, U2.6
- net Split_Comms_TX-A6: now also U2.3, U2.4
- net VCC: now also U2.5; no longer SCREEN1.A4 (VBUS), SCREEN1.A9 (VBUS), SCREEN1.B4 (VBUS), SCREEN1.B9 (VBUS)
