File: mk18-pcb.kicad_sch (KiCad schematic)
At the start: 82 parts, among them P1 FH26W-13S-0_3SHW(60), P10 FH26W-13S-0_3SHW(60), P11 FH26W-13S-0_3SHW(60), P2 FH26W-13S-0_3SHW(60), P3 FH26W-13S-0_3SHW(60), P4 FH26W-13S-0_3SHW(60), P5 FH26W-13S-0_3SHW(60), P6 FH26W-13S-0_3SHW(60), P7 FH26W-13S-0_3SHW(60), P8 FH26W-13S-0_3SHW(60)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

Commit message: final production version of 1.0 woooo
Parts:
- added AUDIO1: Conn_01x03_Socket, Connector_JST:JST_EH_B3B-EH-A_1x03_P2.50mm_Vertical, symbol Connector:Conn_01x03_Socket
- CYBOARD-MACRO1: symbol ct-kicad:HC-FPC-05-10-16RLTAG -> ct-kicad:0_5K-A-16PBF; LCSC C5213735 -> C2914211
- PICO1: now left out of the parts list
Connections:
- net +3V3: now also AUDIO1.3 (Pin_3)
- net GND: now also RESET1.1 (Pin_1), AUDIO1.1 (Pin_1); no longer RESET1.2 (Pin_2)
- net GPIO22: now also AUDIO1.2 (Pin_2)
- net reset: now also RESET1.2 (Pin_2); no longer RESET1.1 (Pin_1)
Other:
- note added: "Audio"
- moved on the sheet: CYBOARD-MACRO1

Commit message: updating readme, tidied up schematic
Parts:
- added LOGO1, LOGO2: **REF, ct-kicad:awesome-logo, symbol ct-kicad:awesome-logo
- added LOGO3, LOGO4: **REF, ct-kicad:qmk-lite, symbol ct-kicad:qmk-lite-logo
Other:
- note added: "5-way breakout"
- note added: "Audio breakout"
- note added: "Breakouts"
- note added: "COL_CS mosfet"
- note added: "Logos"
- note added: "Reference schematics"
- note added: "Row & Col breakouts"
- note removed: "5-way"
- note removed: "Audio"
- moved on the sheet: 5WAY1, ADC1, AUDIO1, C1, C2, C3, C4, C5, C6, COL1, COL2, COL_CS_MOS1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
